File: hardware/eco_measure_v0/wat.kicad_pcb (KiCad board)
At the start: 2 copper layers, 67.9 x 87 mm, 48 parts, among them J1 Conn_02x05_Odd_Even, J2 Conn_01x06, J3 Conn_01x03, J4 Conn_01x06, J5 Conn_01x06, P1 V_IN, U1 NANO

Commit message: raspberry compatible connector
Parts:
- removed J4, J5: Conn_01x06, TerminalBlock:TerminalBlock_bornier-6_P5.08mm
- J2: value Conn_01x06 -> Conn_01x12; footprint TerminalBlock:TerminalBlock_bornier-6_P5.08mm -> eco_power_v2:TerminalBlock_bornier-12_P5.08mm
- J3: value Conn_01x03 -> Conn_01x09; footprint TerminalBlock:TerminalBlock_bornier-3_P5.08mm -> eco_power_v2:TerminalBlock_bornier-9_P5.08mm
- moved J2 30.5 mm to (66.4, 155.0)
- moved J3 10.2 mm to (107.1, 79.2), turned to 180 degrees
Connections:
- J1 pad 10: GND -> Net-(J1-Pad10)
- J1 pad 2: /D6 -> GND
- J2 pad 2: /jA4 -> /jA0
- J2 pad 3: /jA5 -> /jA1
- J2 pad 4: /jA6 -> /jA2
- J2 pad 5: /jA7 -> /jA3
- J3 pad 1: /D3 -> GND
- J3 pad 3: GND -> /D3
- U1 pad 9: /D6 -> Net-(U1-Pad9)
Routing:
- net /D6: track 10.5 -> 0.00 mm
