File: hardware/iot_esp/iotesp_hardware/ecoBeat_3.sch (KiCad schematic (older format))
At the start: 10 parts, among them J1 Test, P1 CONN_02X05, U1 WeMos_mini

Commit message: images to the readme
Parts:
- R8, R9: value 220 -> 1k
Changed lines of the file:
@@
 encoding utf-8
 Sheet 1 1
-Title "Lector de pulsos"
-Date "2018-02-14"
+Title "ecotherm_esp"
+Date "2021-10-24"
 Rev "1"
 Comp ""
@@
 P 8020 3820
 F 0 "R9" V 8100 3820 50  0000 C CNN
-F 1 "220" V 8020 3820 50  0000 C CNN
+F 1 "1k" V 8020 3820 50  0000 C CNN
 F 2 "Resistors_SMD:R_1206_HandSoldering" V 7950 3820 50  0001 C CNN
 F 3 "" H 8020 3820 50  0000 C CNN
@@
 P 8020 3515
 F 0 "R8" V 8100 3515 50  0000 C CNN
-F 1 "220" V 8020 3515 50  0000 C CNN
+F 1 "1k" V 8020 3515 50  0000 C CNN
 F 2 "Resistors_SMD:R_1206_HandSoldering" V 7950 3515 50  0001 C CNN
 F 3 "" H 8020 3515 50  0000 C CNN
